File: free_dry_electrodes_12-18/free_dry_electrodes_12_18.kicad_pcb (KiCad board)
At the start: 2 copper layers, 14 x 14 mm, 30 parts

Commit message: Add files via upload
Parts:
- renumbered REF** to REF1, REF** to REF10, REF** to REF11, REF** to REF12, REF** to REF13, REF** to REF14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
