File: free_dry_electrodes_12_18/free_dry_electrodes_12_18.kicad_sch (KiCad schematic)
At the start: 0 parts

Commit message: Add files via upload
Parts:
- added REF1: CPA_1, symbol Connector_Generic:Conn_01x01
- added REF10, REF11, REF12, REF13, REF14, REF15, REF16, REF17, REF18, REF19, REF2, REF20, REF21, REF22, REF23, REF24, REF25, REF26, REF27, REF28, REF29, REF3, REF30, REF4, REF5, REF6, REF7, REF8, REF9: CPA_1, 1024_dry_electrodes:CPA_1, symbol Connector_Generic:Conn_01x01
Connections:
- new net: REF1.1 (Pin_1), REF10.1 (Pin_1), REF11.1 (Pin_1), REF12.1 (Pin_1), REF13.1 (Pin_1), REF14.1 (Pin_1), REF15.1 (Pin_1), REF16.1 (Pin_1), REF17.1 (Pin_1), REF18.1 (Pin_1), REF19.1 (Pin_1), REF2.1 (Pin_1), REF20.1 (Pin_1), REF21.1 (Pin_1), REF22.1 (Pin_1), REF23.1 (Pin_1), REF24.1 (Pin_1), REF25.1 (Pin_1), REF26.1 (Pin_1), REF27.1 (Pin_1), REF28.1 (Pin_1), REF29.1 (Pin_1), REF3.1 (Pin_1), REF30.1 (Pin_1), REF4.1 (Pin_1), REF5.1 (Pin_1), REF6.1 (Pin_1), REF7.1 (Pin_1), REF8.1 (Pin_1), REF9.1 (Pin_1)
