File: free_dry_electrodes_12_18/free_dry_electrodes_12_18_rectangle.kicad_pcb (KiCad board)
At the start: 2 copper layers, 15.5 x 15.5 mm, 2 parts, among them J1 Conn_01x12, J2 Conn_01x18

Commit message: Add files via upload
Other:
- outline, holes or cut-outs redrawn
Changed lines of the file:
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@@
       (net 1 "Net-(J1-Pad1)") (pinfunction "Pin_12") (pintype "passive"))
   )
+  (gr_circle (center -6.25 -6.25) (end -5.25 -6.25) (layer "Edge.Cuts") (width 0.1) (fill none))
+  (gr_circle (center 6.25 6.25) (end 7.25 6.25) (layer "Edge.Cuts") (width 0.1) (fill none))
+  (gr_circle (center 6.25 -6.25) (end 7.25 -6.25) (layer "Edge.Cuts") (width 0.1) (fill none))
+  (gr_rect (start 7.75 7.75) (end -7.75 -7.75) (layer "Edge.Cuts") (width 0.1) (fill none))
   (gr_circle (center 0 0) (end 3 0) (layer "Edge.Cuts") (width 0.1) (fill none))
-  (gr_circle (center 0 0) (end 7.75 0) (layer "Edge.Cuts") (width 0.1) (fill none))
+  (gr_circle (center -6.25 6.25) (end -5.25 6.25) (layer "Edge.Cuts") (width 0.1) (fill none))
   (segment (start 0 6.5) (end 0 4.25) (width 2) (layer "B.Cu") (net 1))
   (segment (start -2.125 6.009872) (end -2.22313 6.108002) (width 2) (layer "B.Cu") (net 1))
